Commit message: Remove mesh rotation from URDF.

File: urdf/gp7_macro.xacro (robot description, xacro)
@@ -6,5 +6,4 @@
 		<link name="${prefix}base_link">
 			<visual>
-			        <origin rpy="0 0 3.14159"/>
 				<geometry>
 					<mesh filename="package://yaskawa_gp7_support/meshes/gp7/visual/gp7_base_axis.stl" />
@@ -15,5 +14,4 @@
 			</visual>
 			<collision>
-			        <origin rpy="0 0 3.14159"/>
 				<geometry>
 					<mesh filename="package://yaskawa_gp7_support/meshes/gp7/collision/gp7_base_axis.stl" />
@@ -59,5 +57,5 @@
 					<mesh filename="package://yaskawa_gp7_support/meshes/gp7/visual/gp7_u_axis.stl"/>
 				</geometry>
-				<material name="blue"/>
+				<material name="silver"/>
 			</visual>
 			<collision>
@@ -73,5 +71,5 @@
 					<mesh filename="package://yaskawa_gp7_support/meshes/gp7/visual/gp7_r_axis.stl"/>
 				</geometry>
-				<material name="silver"/>
+				<material name="blue"/>
 			</visual>
 			<collision>
@@ -87,5 +85,5 @@
 					<mesh filename="package://yaskawa_gp7_support/meshes/gp7/visual/gp7_b_axis.stl"/>
 				</geometry>
-				<material name="blue"/>
+				<material name="silver"/>
 			</visual>
 			<collision>
@@ -101,5 +99,5 @@
 					<mesh filename="package://yaskawa_gp7_support/meshes/gp7/visual/gp7_t_axis.stl" />
 				</geometry>
-				<material name="silver"/>
+				<material name="blue"/>
 			</visual>
 			<collision>

Commit message: Add flange frame.

File: urdf/gp7_macro.xacro (robot description, xacro)
@@ -108,4 +108,5 @@
 			</collision>
 		</link>
+		<link name="${prefix}flange" />
 		<!-- end of link list -->
 		<!-- joint list -->
@@ -152,4 +153,9 @@
 			<limit lower="${-360 * pi / 180}" upper="${360 * pi / 180}" effort="1" velocity="${1000 * pi / 180}" />
 		</joint>
+		<joint name="${prefix}joint_flange" type="fixed">
+			<parent link="${prefix}link_t"/>
+			<child link="${prefix}flange"/>
+			<origin rpy="0 ${-0.5 * pi} ${pi}"/>
+		</joint>
 		<!-- end of joint list -->
 	</xacro:macro>

Commit message: Add vendor_base_link.

File: urdf/gp7_macro.xacro (robot description, xacro)
@@ -22,4 +22,5 @@
 			</collision>
 		</link>
+		<link name="${prefix}vendor_base_link" />
 		<link name="${prefix}link_s">
 			<visual>
@@ -109,5 +110,4 @@
 		</link>
 		<link name="${prefix}flange" />
-		<!-- end of link list -->
 		<!-- joint list -->
 		<joint name="${prefix}joint_s" type="revolute">
@@ -117,4 +117,9 @@
 			<axis xyz="0 0 1" />
 			<limit lower="${-170 * pi / 180}" upper="${170 * pi / 180}" effort="1" velocity="${375 * pi / 180}" />
+		</joint>
+		<joint name="${prefix}joint_vendor_base" type="fixed">
+			<parent link="${prefix}base_link"/>
+			<child link="${prefix}vendor_base_link"/>
+			<origin xyz="0 0 0.330" />
 		</joint>
 		<joint name="${prefix}joint_l" type="revolute">
@@ -158,5 +163,4 @@
 			<origin rpy="0 ${-0.5 * pi} ${pi}"/>
 		</joint>
-		<!-- end of joint list -->
 	</xacro:macro>
 </robot>
